File: hardware/NosVolt.kicad_sch (KiCad schematic)
At the start: 19 parts, among them J1 USB_C_Receptacle_USB2.0_16P, SW1 SW_Reset, U1 USBLC6-2SC6, U2 AP7361-33ER-13, U3 ESP32-S3-WROOM-1

Commit message: ldo
Parts:
- removed C1: 1nF, Capacitor_SMD:C_0805_2012Metric, symbol Device:C
- removed C3, C5: 100nF, Capacitor_SMD:C_0603_1608Metric, symbol Device:C
- removed C4, C6: 10uF, Capacitor_SMD:C_0805_2012Metric, symbol Device:C
- removed D1: SMBJ5.0A, Diode_SMD:D_SMB, symbol Device:D_Zener
- removed F1: Polyfuse, Fuse:Fuse_0805_2012Metric, symbol Device:Polyfuse
- removed J1: USB_C_Receptacle_USB2.0_16P, Connector_USB:USB_C_Receptacle_HRO_TYPE-C-31-M-12, symbol Connector:USB_C_Receptacle_USB2.0_16P
- removed R5, R6: 5.1K, Resistor_SMD:R_0603_1608Metric, symbol Device:R
- removed U1: USBLC6-2SC6, Package_TO_SOT_SMD:SOT-23-6, symbol Power_Protection:USBLC6-2SC6
- removed U2: AP7361-33ER-13, Package_TO_SOT_SMD:SOT-223-3_TabPin2, symbol Regulator_Linear:AMS1117-3.3
- added SW2: MSK-12D19, symbol Switch:SW_SPDT
- SW1: footprint Button_Switch_THT:SW_PUSH_6mm_H4.3mm -> Button_Switch_SMD:SW_Push_SPST_NO_Alps_SKRK
Connections:
- net +3.3V: now also SW2.2 (B)
- new net MP2307/OUT: SW2.1 (A)
- new net USB_LDO/3V3: SW2.3 (C)
- no-connect marks 2 -> 0
Other:
- added sheet USB_LDO (USB_LDO.kicad_sch)
- sheet MP2307 ports: added IN, OUT; removed none

Commit message: Outputs and current measurement
Parts:
- added J101: IN, TerminalBlock_Phoenix:TerminalBlock_Phoenix_MKDS-1,5-2-5.08_1x02_P5.08mm_Horizontal, symbol Connector:Screw_Terminal_01x02
- added J102: BAT, TerminalBlock_Phoenix:TerminalBlock_Phoenix_MKDS-1,5-2-5.08_1x02_P5.08mm_Horizontal, symbol Connector:Screw_Terminal_01x02
- added J103: INT_OUT, TerminalBlock_Phoenix:TerminalBlock_Phoenix_MKDS-1,5-2-5.08_1x02_P5.08mm_Horizontal, symbol Connector:Screw_Terminal_01x02
- added J104: OUT1, TerminalBlock_Phoenix:TerminalBlock_Phoenix_MKDS-1,5-2-5.08_1x02_P5.08mm_Horizontal, symbol Connector:Screw_Terminal_01x02
- added J105: OUT2, TerminalBlock_Phoenix:TerminalBlock_Phoenix_MKDS-1,5-2-5.08_1x02_P5.08mm_Horizontal, symbol Connector:Screw_Terminal_01x02
- added J106: OUT3, TerminalBlock_Phoenix:TerminalBlock_Phoenix_MKDS-1,5-2-5.08_1x02_P5.08mm_Horizontal, symbol Connector:Screw_Terminal_01x02
- R101: renamed from R1; footprint Resistor_SMD:R_0603_1608Metric -> Resistor_SMD:R_0603_1608Metric_Pad0.98x0.95mm_HandSolder
- R102: renamed from R4; footprint Resistor_SMD:R_0603_1608Metric -> Resistor_SMD:R_0603_1608Metric_Pad0.98x0.95mm_HandSolder
- R103: renamed from R2; footprint Resistor_SMD:R_0603_1608Metric -> Resistor_SMD:R_0603_1608Metric_Pad0.98x0.95mm_HandSolder
- R104: renamed from R3; footprint Resistor_SMD:R_0603_1608Metric -> Resistor_SMD:R_0603_1608Metric_Pad0.98x0.95mm_HandSolder
- SW102: renamed from SW2; value MSK-12D19 -> SSSS811101; footprint (none) -> SSSS811101:SW_SSSS811101; symbol Switch:SW_SPDT -> NosLib:SSSS811101
- renumbered C2 to C101, SW1 to SW101, U3 to U101
Connections:
- net +12V_UPS: now also J103.1 (Pin_1)
- net +3.3V: no longer SW102.2 (B)
- net GND: now also SW102.SH1 (SH), SW102.SH2 (SH), SW102.SH3 (SH), SW102.SH4 (SH), J103.2 (Pin_2), J104.2 (Pin_2), J105.2 (Pin_2), J106.2 (Pin_2)
- net MP2307/OUT: now also SW102.3; no longer SW102.1 (A)
- net USB_LDO/3V3: now also SW102.1; no longer SW102.3 (C)
- net EN_OUT1: now reaches U101.4 (GPIO4/TOUCH4/ADC1_CH3)
- net EN_OUT2: now reaches U101.5 (GPIO5/TOUCH5/ADC1_CH4)
- net EN_OUT3: now reaches U101.6 (GPIO6/TOUCH6/ADC1_CH5)
- new net INA226_BAT/VIN+: J102.1 (Pin_1)
- new net INA226_BAT/VIN-: J102.2 (Pin_2)
- new net INA226_IN/VIN+: J101.1 (Pin_1)
- new net INA226_IN/VIN-: J101.2 (Pin_2)
- new net Output1/VOUT: J104.1 (Pin_1)
- new net Output2/VOUT: J105.1 (Pin_1)
- new net Output3/VOUT: J106.1 (Pin_1)
Other:
- added sheet INA226_BAT (INA226.kicad_sch)
- added sheet INA226_IN (INA226.kicad_sch)
- added sheet Output1 (Output.kicad_sch)
- added sheet Output2 (Output.kicad_sch)
- added sheet Output3 (Output.kicad_sch)
- note added: "ESP32 EN, BOOT, I2C"
- note added: "Power Supply"
- moved on the sheet: R101, R103, R104, U101

Commit message: Tracing 1
Parts:
- removed J101: IN, TerminalBlock_Phoenix:TerminalBlock_Phoenix_MKDS-1,5-2-5.08_1x02_P5.08mm_Horizontal, symbol Connector:Screw_Terminal_01x02
- removed J102: BAT, TerminalBlock_Phoenix:TerminalBlock_Phoenix_MKDS-1,5-2-5.08_1x02_P5.08mm_Horizontal, symbol Connector:Screw_Terminal_01x02
- removed J103: INT_OUT, TerminalBlock_Phoenix:TerminalBlock_Phoenix_MKDS-1,5-2-5.08_1x02_P5.08mm_Horizontal, symbol Connector:Screw_Terminal_01x02
- removed J104: OUT1, TerminalBlock_Phoenix:TerminalBlock_Phoenix_MKDS-1,5-2-5.08_1x02_P5.08mm_Horizontal, symbol Connector:Screw_Terminal_01x02
- removed J105: OUT2, TerminalBlock_Phoenix:TerminalBlock_Phoenix_MKDS-1,5-2-5.08_1x02_P5.08mm_Horizontal, symbol Connector:Screw_Terminal_01x02
- removed J106: OUT3, TerminalBlock_Phoenix:TerminalBlock_Phoenix_MKDS-1,5-2-5.08_1x02_P5.08mm_Horizontal, symbol Connector:Screw_Terminal_01x02
- added J101: OUTPUTS, TerminalBlock_Phoenix:TerminalBlock_Phoenix_MKDS-1,5-6-5.08_1x06_P5.08mm_Horizontal, symbol Connector:Screw_Terminal_01x06
- added J107: INPUTS, TerminalBlock_Phoenix:TerminalBlock_Phoenix_MKDS-1,5-6-5.08_1x06_P5.08mm_Horizontal, symbol Connector:Screw_Terminal_01x06
Connections:
- net +12V_UPS: now also J107.5 (Pin_5)
- net GND: now also J101.2 (Pin_2), J101.4 (Pin_4), J101.6 (Pin_6), J107.6 (Pin_6)
- net INA226_BAT/VIN+: now also J107.3 (Pin_3)
- net INA226_BAT/VIN-: now also J107.4 (Pin_4)
- net INA226_IN/VIN+: now also J107.1 (Pin_1)
- net INA226_IN/VIN-: now also J107.2 (Pin_2)
- net Output1/VOUT: now also J101.1 (Pin_1)
- net Output2/VOUT: now also J101.3 (Pin_3)
- net Output3/VOUT: now also J101.5 (Pin_5)

Commit message: Tracing 2
Connections:
- net INA226_BAT/VIN+ renamed INA226_BAT/VOUT
- net INA226_BAT/VIN- renamed INA226_BAT/VIN
- net INA226_IN/VIN+ renamed INA226_IN/VOUT
- net INA226_IN/VIN- renamed INA226_IN/VIN
Other:
- sheet INA226_BAT ports: added VIN, VOUT; removed VIN+, VIN-
- sheet INA226_IN ports: added VIN, VOUT; removed VIN+, VIN-
Changed lines of the file:
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@@
 	(wire
 		(pts
+			(xy 26.67 124.46) (xy 41.91 124.46)
+		)
+		(stroke
+			(width 0)
+			(type default)
+		)
+	)
+	(wire
+		(pts
 			(xy 88.9 147.32) (xy 104.14 147.32)
 		)
@@
 	(wire
 		(pts
-			(xy 25.4 151.13) (xy 25.4 121.92)
+			(xy 102.87 127) (xy 104.14 127)
 		)
 		(stroke
@@
 	(wire
 		(pts
-			(xy 102.87 127) (xy 104.14 127)
+			(xy 152.4 128.27) (xy 152.4 148.59)
 		)
 		(stroke
@@
 	(wire
 		(pts
-			(xy 154.94 125.73) (xy 154.94 146.05)
-		)
-		(stroke
-			(width 0)
-			(type default)
-		)
-	)
-	(wire
-		(pts
 			(xy 82.55 147.32) (xy 88.9 147.32)
 		)
@@
 	(wire
 		(pts
-			(xy 30.48 158.75) (xy 30.48 144.78)
+			(xy 25.4 121.92) (xy 25.4 151.13)
 		)
 		(stroke
@@
 	(wire
 		(pts
-			(xy 30.48 144.78) (xy 41.91 144.78)
+			(xy 30.48 158.75) (xy 30.48 144.78)
 		)
 		(stroke
@@
 	(wire
 		(pts
-			(xy 152.4 148.59) (xy 160.02 148.59)
-		)
-		(stroke
-			(width 0)
-			(type default)
-		)
-	)
-	(wire
-		(pts
 			(xy 67.31 147.32) (xy 82.55 147.32)
 		)
@@
 	(wire
 		(pts
-			(xy 26.67 124.46) (xy 26.67 153.67)
-		)
-		(stroke
-			(width 0)
-			(type default)
-		)
-	)
-	(wire
-		(pts
 			(xy 69.85 163.83) (xy 69.85 149.86)
 		)
@@
 	(wire
 		(pts
-			(xy 26.67 124.46) (xy 41.91 124.46)
+			(xy 130.81 125.73) (xy 154.94 125.73)
 		)
 		(stroke
@@
 	(wire
 		(pts
-			(xy 130.81 125.73) (xy 154.94 125.73)
+			(xy 55.88 82.55) (xy 62.23 82.55)
 		)
 		(stroke
@@
 	(wire
 		(pts
-			(xy 55.88 82.55) (xy 62.23 82.55)
+			(xy 154.94 146.05) (xy 160.02 146.05)
 		)
 		(stroke
@@
 	(wire
 		(pts
+			(xy 152.4 148.59) (xy 160.02 148.59)
+		)
+		(stroke
+			(width 0)
+			(type default)
+		)
+	)
+	(wire
+		(pts
 			(xy 57.15 46.99) (xy 69.85 46.99)
 		)
@@
 	(wire
 		(pts
-			(xy 154.94 146.05) (xy 160.02 146.05)
+			(xy 57.15 36.83) (xy 57.15 35.56)
 		)
 		(stroke
@@
 	(wire
 		(pts
-			(xy 57.15 36.83) (xy 57.15 35.56)
+			(xy 88.9 121.92) (xy 104.14 121.92)
 		)
 		(stroke
@@
 	(wire
 		(pts
-			(xy 88.9 121.92) (xy 104.14 121.92)
+			(xy 154.94 125.73) (xy 154.94 146.05)
 		)
 		(stroke
@@
 	(wire
 		(pts
-			(xy 29.21 142.24) (xy 41.91 142.24)
+			(xy 91.44 36.83) (xy 91.44 40.64)
 		)
 		(stroke
@@
 	(wire
 		(pts
-			(xy 152.4 128.27) (xy 152.4 148.59)
+			(xy 154.94 158.75) (xy 160.02 158.75)
 		)
 		(stroke
@@
 	(wire
 		(pts
-			(xy 91.44 36.83) (xy 91.44 40.64)
+			(xy 26.67 124.46) (xy 26.67 153.67)
 		)
 		(stroke
@@
 	(wire
 		(pts
-			(xy 154.94 158.75) (xy 160.02 158.75)
+			(xy 102.87 176.53) (xy 104.14 176.53)
 		)
 		(stroke
@@
 	(wire
 		(pts
-			(xy 102.87 176.53) (xy 104.14 176.53)
+			(xy 30.48 144.78) (xy 41.91 144.78)
 		)
 		(stroke
@@
 		)
 	)
+	(wire
+		(pts
+			(xy 29.21 142.24) (xy 41.91 142.24)
+		)
+		(stroke
+			(width 0)
+			(type default)
+		)
+	)
 	(global_label "BOOT"
 		(shape input)
@@
 			)
 		)
-		(pin "VIN+" input
-			(at 41.91 121.92 180)
+		(pin "A1" input
+			(at 41.91 129.54 180)
 			(effects
 				(font
@@
 			)
 		)
-		(pin "A1" input
-			(at 41.91 129.54 180)
+		(pin "A0" input
+			(at 41.91 127 180)
 			(effects
 				(font
@@
 			)
 		)
-		(pin "VIN-" input
+		(pin "VIN" input
 			(at 41.91 124.46 180)
 			(effects
@@
 			)
 		)
-		(pin "A0" input
-			(at 41.91 127 180)
+		(pin "VOUT" input
+			(at 41.91 121.92 180)
 			(effects
 				(font
@@
 			)
 		)
-		(pin "VIN+" input
-			(at 41.91 142.24 180)
+		(pin "A1" input
+			(at 41.91 149.86 180)
 			(effects
 				(font
@@
 			)
 		)
-		(pin "A1" input
-			(at 41.91 149.86 180)
+		(pin "A0" input
+			(at 41.91 147.32 180)
 			(effects
 				(font
@@
 			)
 		)
-		(pin "VIN-" input
+		(pin "VIN" input
 			(at 41.91 144.78 180)
 			(effects
@@
 			)
 		)
-		(pin "A0" input
-			(at 41.91 147.32 180)
+		(pin "VOUT" input
+			(at 41.91 142.24 180)
 			(effects
 				(font
