File: hardware/NosVolt.kicad_pcb (KiCad board)
At the start: 2 copper layers, 48 parts, among them J1 USB_C_Receptacle_USB2.0_16P, J2 BAT_SENSE, SW1 SW_Reset, U1 USBLC6-2SC6, U2 AP7361-33ER-13, U3 ESP32-S3-WROOM-1, U4 ADS1115IDGS, U5 MP2307DN-LF-Z

Commit message: Outputs and current measurement
Parts:
- removed C1: 1nF, Capacitor_SMD:C_0805_2012Metric
- removed C3, C5: 100nF, Capacitor_SMD:C_0603_1608Metric
- removed C4, C6: 10uF, Capacitor_SMD:C_0805_2012Metric
- removed D1: SMBJ5.0A, Diode_SMD:D_SMB
- removed F1: Polyfuse, Fuse:Fuse_0805_2012Metric
- removed J1: USB_C_Receptacle_USB2.0_16P, Connector_USB:USB_C_Receptacle_HRO_TYPE-C-31-M-12
- removed R5, R6: 5.1K, Resistor_SMD:R_0603_1608Metric
- removed U1: USBLC6-2SC6, Package_TO_SOT_SMD:SOT-23-6
- removed U2: AP7361-33ER-13, Package_TO_SOT_SMD:SOT-223-3_TabPin2
- added C1001: 100nF, Capacitor_SMD:C_0603_1608Metric, F.Cu at (46.6, 96.3)
- added C1002: 100nF, Capacitor_SMD:C_0603_1608Metric, F.Cu at (46.6, 98.8)
- added C1101: 22nF, Capacitor_SMD:C_0805_2012Metric, F.Cu at (59.1, 43.4)
- added C1102: 100nF, Capacitor_SMD:C_0603_1608Metric, F.Cu at (54.5, 46.6)
- added C1103: 22uF, Capacitor_SMD:C_0805_2012Metric, F.Cu at (59.1, 46.4)
- added C1201: 100nF, Capacitor_SMD:C_0603_1608Metric, F.Cu at (43.5, 46.0)
- added C1202: 100nF, Capacitor_SMD:C_0603_1608Metric, F.Cu at (43.5, 48.5)
- added C401: 1nF, Capacitor_SMD:C_0805_2012Metric, F.Cu at (217.2, 75.3)
- added C402: 100nF, Capacitor_SMD:C_0603_1608Metric, F.Cu at (228.6, 64.6)
- added C403: 10uF, Capacitor_SMD:C_0805_2012Metric, F.Cu at (217.2, 78.3)
- added C404: 100nF, Capacitor_SMD:C_0603_1608Metric, F.Cu at (228.6, 67.1)
- added C405: 10uF, Capacitor_SMD:C_0805_2012Metric, F.Cu at (217.2, 81.3)
- added C501: 100nF, Capacitor_SMD:C_0603_1608Metric, F.Cu at (102.6, 72.2)
- added C502: 100nF, Capacitor_SMD:C_0603_1608Metric, F.Cu at (102.6, 74.7)
- added C601: 100nF, Capacitor_SMD:C_0603_1608Metric, F.Cu at (126.7, 96.1)
- added C602: 100nF, Capacitor_SMD:C_0603_1608Metric, F.Cu at (126.7, 98.7)
- added C701: 100nF, Capacitor_SMD:C_0603_1608Metric, F.Cu at (163.8, 94.6)
- added C702: 100nF, Capacitor_SMD:C_0603_1608Metric, F.Cu at (163.8, 97.1)
- added C801: 22nF, Capacitor_SMD:C_0805_2012Metric, F.Cu at (125.3, 59.8)
- added C802: 100nF, Capacitor_SMD:C_0603_1608Metric, F.Cu at (134.3, 46.4)
- added C803: 22uF, Capacitor_SMD:C_0805_2012Metric, F.Cu at (139.0, 50.6)
- added C901: 22nF, Capacitor_SMD:C_0805_2012Metric, F.Cu at (51.1, 110.2)
- added C902: 100nF, Capacitor_SMD:C_0603_1608Metric, F.Cu at (46.6, 113.4)
- added C903: 22uF, Capacitor_SMD:C_0805_2012Metric, F.Cu at (51.1, 113.2)
- added D401: SMF5.0A, Diode_SMD:D_SMF, F.Cu at (232.2, 80.1)
- added F401: Polyfuse 0.75A, Fuse:Fuse_0805_2012Metric, F.Cu at (232.9, 64.8)
- added J101: IN, TerminalBlock_Phoenix:TerminalBlock_Phoenix_MKDS-1,5-2-5.08_1x02_P5.08mm_Horizontal, F.Cu at (118.4, 90.6)
- added J102: BAT, TerminalBlock_Phoenix:TerminalBlock_Phoenix_MKDS-1,5-2-5.08_1x02_P5.08mm_Horizontal, F.Cu at (131.2, 61.4)
- added J103: INT_OUT, TerminalBlock_Phoenix:TerminalBlock_Phoenix_MKDS-1,5-2-5.08_1x02_P5.08mm_Horizontal, F.Cu at (167.5, 75.0)
- added J104: OUT1, TerminalBlock_Phoenix:TerminalBlock_Phoenix_MKDS-1,5-2-5.08_1x02_P5.08mm_Horizontal, F.Cu at (99.2, 53.6)
- added J105: OUT2, TerminalBlock_Phoenix:TerminalBlock_Phoenix_MKDS-1,5-2-5.08_1x02_P5.08mm_Horizontal, F.Cu at (29.2, 82.0)
- added J106: OUT3, TerminalBlock_Phoenix:TerminalBlock_Phoenix_MKDS-1,5-2-5.08_1x02_P5.08mm_Horizontal, F.Cu at (27.8, 42.1)
- added J401: USB_C_Receptacle_USB2.0_16P, Connector_USB:USB_C_Receptacle_HRO_TYPE-C-31-M-12, F.Cu at (203.0, 52.9)
- added Q1101: 2N7002, Package_TO_SOT_SMD:SOT-23, F.Cu at (63.8, 44.1)
- added Q1102: AO4407A, Package_SO:SOIC-8_3.9x4.9mm_P1.27mm, F.Cu at (61.1, 38.6)
- added Q801: 2N7002, Package_TO_SOT_SMD:SOT-23, F.Cu at (139.7, 44.2)
- added Q802: AO4407A, Package_SO:SOIC-8_3.9x4.9mm_P1.27mm, F.Cu at (126.8, 46.9)
- added Q901: 2N7002, Package_TO_SOT_SMD:SOT-23, F.Cu at (55.8, 110.9)
- added Q902: AO4407A, Package_SO:SOIC-8_3.9x4.9mm_P1.27mm, F.Cu at (53.1, 105.4)
- added R1001: 0.01R, Resistor_SMD:R_2512_6332Metric_Pad1.40x3.35mm_HandSolder, F.Cu at (49.1, 88.0)
- added R1002: 10R, Resistor_SMD:R_0603_1608Metric_Pad0.98x0.95mm_HandSolder, F.Cu at (50.7, 96.3)
- added R1003: 10R, Resistor_SMD:R_0603_1608Metric_Pad0.98x0.95mm_HandSolder, F.Cu at (50.7, 98.8)
- added R1101: 1K, Resistor_SMD:R_0603_1608Metric_Pad0.98x0.95mm_HandSolder, F.Cu at (54.7, 36.5)
- added R1102: 100K, Resistor_SMD:R_0603_1608Metric_Pad0.98x0.95mm_HandSolder, F.Cu at (54.7, 39.1)
- added R1103: 100K, Resistor_SMD:R_0603_1608Metric_Pad0.98x0.95mm_HandSolder, F.Cu at (54.7, 41.6)
- added R1104: 47R, Resistor_SMD:R_0603_1608Metric_Pad0.98x0.95mm_HandSolder, F.Cu at (54.7, 44.1)
- added R1201: 0.01R, Resistor_SMD:R_2512_6332Metric_Pad1.40x3.35mm_HandSolder, F.Cu at (46.0, 37.7)
- added R1202: 10R, Resistor_SMD:R_0603_1608Metric_Pad0.98x0.95mm_HandSolder, F.Cu at (47.6, 46.0)
- added R1203: 10R, Resistor_SMD:R_0603_1608Metric_Pad0.98x0.95mm_HandSolder, F.Cu at (47.6, 48.5)
- added R401: 5.1K, Resistor_SMD:R_0603_1608Metric_Pad0.98x0.95mm_HandSolder, F.Cu at (228.6, 69.6)
- added R402: 5.1K, Resistor_SMD:R_0603_1608Metric_Pad0.98x0.95mm_HandSolder, F.Cu at (228.6, 72.1)
- added R501: 0.01R, Resistor_SMD:R_2512_6332Metric_Pad1.40x3.35mm_HandSolder, F.Cu at (105.1, 63.9)
- added R502: 10R, Resistor_SMD:R_0603_1608Metric_Pad0.98x0.95mm_HandSolder, F.Cu at (106.8, 72.2)
- added R503: 10R, Resistor_SMD:R_0603_1608Metric_Pad0.98x0.95mm_HandSolder, F.Cu at (106.8, 74.7)
- added R601: 0.01R, Resistor_SMD:R_2512_6332Metric_Pad1.40x3.35mm_HandSolder, F.Cu at (129.2, 87.9)
- added R602: 10R, Resistor_SMD:R_0603_1608Metric_Pad0.98x0.95mm_HandSolder, F.Cu at (130.9, 96.1)
- added R603: 10R, Resistor_SMD:R_0603_1608Metric_Pad0.98x0.95mm_HandSolder, F.Cu at (130.9, 98.7)
- added R701: 0.01R, Resistor_SMD:R_2512_6332Metric_Pad1.40x3.35mm_HandSolder, F.Cu at (166.3, 86.3)
- added R702: 10R, Resistor_SMD:R_0603_1608Metric_Pad0.98x0.95mm_HandSolder, F.Cu at (168.0, 94.6)
- added R703: 10R, Resistor_SMD:R_0603_1608Metric_Pad0.98x0.95mm_HandSolder, F.Cu at (168.0, 97.1)
- added R801: 1K, Resistor_SMD:R_0603_1608Metric_Pad0.98x0.95mm_HandSolder, F.Cu at (120.9, 53.0)
- added R802: 100K, Resistor_SMD:R_0603_1608Metric_Pad0.98x0.95mm_HandSolder, F.Cu at (120.9, 55.5)
- added R803: 100K, Resistor_SMD:R_0603_1608Metric_Pad0.98x0.95mm_HandSolder, F.Cu at (120.9, 58.0)
- added R804: 47R, Resistor_SMD:R_0603_1608Metric_Pad0.98x0.95mm_HandSolder, F.Cu at (120.9, 60.5)
- added R901: 1K, Resistor_SMD:R_0603_1608Metric_Pad0.98x0.95mm_HandSolder, F.Cu at (46.7, 103.3)
- added R902: 100K, Resistor_SMD:R_0603_1608Metric_Pad0.98x0.95mm_HandSolder, F.Cu at (46.7, 105.8)
- added R903: 100K, Resistor_SMD:R_0603_1608Metric_Pad0.98x0.95mm_HandSolder, F.Cu at (46.7, 108.3)
- added R904: 47R, Resistor_SMD:R_0603_1608Metric_Pad0.98x0.95mm_HandSolder, F.Cu at (46.7, 110.9)
- added SW102: SSSS811101, SSSS811101:SW_SSSS811101, F.Cu at (166.6, 48.7)
- added U1001: INA226, Package_SO:VSSOP-10_3x3mm_P0.5mm, F.Cu at (48.3, 92.8)
- added U1201: INA226, Package_SO:VSSOP-10_3x3mm_P0.5mm, F.Cu at (45.2, 42.5)
- added U401: AP7361-33ER-13, Package_TO_SOT_SMD:SOT-223-3_TabPin2, F.Cu at (224.3, 78.0)
- added U402: USBLC6-2SC6, Package_TO_SOT_SMD:SOT-23-6, F.Cu at (231.8, 76.2)
- added U501: INA226, Package_SO:VSSOP-10_3x3mm_P0.5mm, F.Cu at (104.3, 68.7)
- added U601: INA226, Package_SO:VSSOP-10_3x3mm_P0.5mm, F.Cu at (128.4, 92.6)
- added U701: INA226, Package_SO:VSSOP-10_3x3mm_P0.5mm, F.Cu at (165.5, 91.0)
- R101: renamed from R1; footprint Resistor_SMD:R_0603_1608Metric -> Resistor_SMD:R_0603_1608Metric_Pad0.98x0.95mm_HandSolder
- R102: renamed from R4; footprint Resistor_SMD:R_0603_1608Metric -> Resistor_SMD:R_0603_1608Metric_Pad0.98x0.95mm_HandSolder
- R103: renamed from R2; footprint Resistor_SMD:R_0603_1608Metric -> Resistor_SMD:R_0603_1608Metric_Pad0.98x0.95mm_HandSolder
- R104: renamed from R3; footprint Resistor_SMD:R_0603_1608Metric -> Resistor_SMD:R_0603_1608Metric_Pad0.98x0.95mm_HandSolder
- R201: renamed from R7; footprint Resistor_SMD:R_0603_1608Metric -> Resistor_SMD:R_0603_1608Metric_Pad0.98x0.95mm_HandSolder
- R202: renamed from R8; footprint Resistor_SMD:R_0603_1608Metric -> Resistor_SMD:R_0603_1608Metric_Pad0.98x0.95mm_HandSolder
- R203: renamed from R9; footprint Resistor_SMD:R_0603_1608Metric -> Resistor_SMD:R_0603_1608Metric_Pad0.98x0.95mm_HandSolder
- R204: renamed from R10; footprint Resistor_SMD:R_0603_1608Metric -> Resistor_SMD:R_0603_1608Metric_Pad0.98x0.95mm_HandSolder
- R205: renamed from R11; footprint Resistor_SMD:R_0603_1608Metric -> Resistor_SMD:R_0603_1608Metric_Pad0.98x0.95mm_HandSolder
- R206: renamed from R12; footprint Resistor_SMD:R_0603_1608Metric -> Resistor_SMD:R_0603_1608Metric_Pad0.98x0.95mm_HandSolder
- R207: renamed from R13; footprint Resistor_SMD:R_0603_1608Metric -> Resistor_SMD:R_0603_1608Metric_Pad0.98x0.95mm_HandSolder
- R301: renamed from R14; footprint Resistor_SMD:R_0603_1608Metric -> Resistor_SMD:R_0603_1608Metric_Pad0.98x0.95mm_HandSolder
- R302: renamed from R15; footprint Resistor_SMD:R_0603_1608Metric -> Resistor_SMD:R_0603_1608Metric_Pad0.98x0.95mm_HandSolder
- R303: renamed from R16; footprint Resistor_SMD:R_0603_1608Metric -> Resistor_SMD:R_0603_1608Metric_Pad0.98x0.95mm_HandSolder
- R304: renamed from R17; footprint Resistor_SMD:R_0603_1608Metric -> Resistor_SMD:R_0603_1608Metric_Pad0.98x0.95mm_HandSolder
- SW101: renamed from SW1; footprint Button_Switch_THT:SW_PUSH_6mm_H4.3mm -> Button_Switch_SMD:SW_Push_SPST_NO_Alps_SKRK
- U301: renamed from U5; footprint Package_SO:SOIC-8-1EP_3.9x4.9mm_P1.27mm_EP2.29x3mm_ThermalVias -> Package_SO:SOIC-8-1EP_3.9x4.9mm_P1.27mm_EP2.29x3mm
- moved C301 115.4 mm to (137.8, 132.4)
- moved C302 115.4 mm to (140.8, 132.4)
- moved C306 115.4 mm to (145.8, 137.4)
- moved C307 115.4 mm to (148.3, 137.4)
- moved R304 115.4 mm to (154.3, 141.2)
- moved C305 115.4 mm to (139.9, 128.5)
- moved R301 115.4 mm to (155.5, 131.0)
- moved R302 115.4 mm to (159.6, 133.5)
- moved R303 115.4 mm to (155.1, 137.5)
- moved C303 115.4 mm to (155.5, 128.0)
- moved C304 115.4 mm to (155.3, 133.5)
- moved L301 115.4 mm to (138.8, 138.7)
- moved NT201 115.4 mm to (167.3, 147.5)
- moved U301 115.4 mm to (146.9, 131.7)
- moved SW101 111.0 mm to (218.8, 130.3)
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- renumbered C2 to C101, C7 to C201, C8 to C202, C9 to C203, C10 to C204, C11 to C205, C12 to C206, C13 to C301, C14 to C302, C15 to C303, C16 to C304, C17 to C305, C18 to C306, C19 to C307, J2 to J201, L1 to L301, NT1 to NT201, U3 to U101, U4 to U201
Connections:
- net +3.3V_UPS renamed /MP2307/OUT
- U101 pad 4: unconnected-(U3-GPIO4/TOUCH4/ADC1_CH3-Pad4) -> EN_OUT1
- U101 pad 5: unconnected-(U3-GPIO5/TOUCH5/ADC1_CH4-Pad5) -> EN_OUT2
- U101 pad 6: unconnected-(U3-GPIO6/TOUCH6/ADC1_CH5-Pad6) -> EN_OUT3
Other:
- copper layers 2 -> 4

Commit message: Tracing 1
Parts:
- removed J102: BAT, TerminalBlock_Phoenix:TerminalBlock_Phoenix_MKDS-1,5-2-5.08_1x02_P5.08mm_Horizontal
- removed J103: INT_OUT, TerminalBlock_Phoenix:TerminalBlock_Phoenix_MKDS-1,5-2-5.08_1x02_P5.08mm_Horizontal
- removed J104: OUT1, TerminalBlock_Phoenix:TerminalBlock_Phoenix_MKDS-1,5-2-5.08_1x02_P5.08mm_Horizontal
- removed J105: OUT2, TerminalBlock_Phoenix:TerminalBlock_Phoenix_MKDS-1,5-2-5.08_1x02_P5.08mm_Horizontal
- removed J106: OUT3, TerminalBlock_Phoenix:TerminalBlock_Phoenix_MKDS-1,5-2-5.08_1x02_P5.08mm_Horizontal
- removed NT201: BAT_0-GND, NetTie:NetTie-2_SMD_Pad0.5mm
- added J107: INPUTS, TerminalBlock_Phoenix:TerminalBlock_Phoenix_MKDS-1,5-6-5.08_1x06_P5.08mm_Horizontal, F.Cu at (56.7, 64.5)
- J101: value IN -> OUTPUTS; footprint TerminalBlock_Phoenix:TerminalBlock_Phoenix_MKDS-1,5-2-5.08_1x02_P5.08mm_Horizontal -> TerminalBlock_Phoenix:TerminalBlock_Phoenix_MKDS-1,5-6-5.08_1x06_P5.08mm_Horizontal
- moved R1001 112.7 mm to (153.2, 131.3)
- moved R1002 112.7 mm to (154.8, 139.5)
- moved C1001 112.7 mm to (150.7, 139.5)
- moved C1002 112.7 mm to (150.7, 142.0)
- moved C902 112.7 mm to (150.7, 156.6)
- moved Q901 112.7 mm to (159.9, 154.1)
- moved R1003 112.7 mm to (154.8, 142.0)
- moved C901 112.7 mm to (155.2, 153.4)
- moved C903 112.7 mm to (155.2, 156.4)
- moved Q902 112.7 mm to (157.2, 148.7)
- moved R901 112.7 mm to (150.8, 146.6)
- moved R902 112.7 mm to (150.8, 149.1)
- moved R903 112.7 mm to (150.8, 151.6)
- moved R904 112.7 mm to (150.8, 154.1)
- moved U1001 112.7 mm to (152.4, 136.0)
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Connections:
- net Net-(F401-Pad1) renamed /USB_LDO/RAW_5V
- J101 pad 1: /INA226_IN/VIN+ -> /Output1/VOUT
- J101 pad 2: /INA226_IN/VIN- -> GND
- J401 pad A6: Net-(J401-D+-PadA6) -> /USB_LDO/RAW_USB_D+
- J401 pad A7: Net-(J401-D--PadA7) -> /USB_LDO/RAW_USB_D-
- J401 pad B6: Net-(J401-D+-PadA6) -> /USB_LDO/RAW_USB_D+
- J401 pad B7: Net-(J401-D--PadA7) -> /USB_LDO/RAW_USB_D-
- U402 pad 1: USB_D- -> /USB_LDO/RAW_USB_D-
- U402 pad 3: USB_D+ -> /USB_LDO/RAW_USB_D+
- U402 pad 4: Net-(J401-D+-PadA6) -> USB_D+
- U402 pad 6: Net-(J401-D--PadA7) -> USB_D-
Routing:
- net /USB_LDO/5V: track 0.00 -> 23.9 mm
- net Net-(J401-SHIELD): track 0.00 -> 23.4 mm
- net /USB_LDO/3V3: track 0.00 -> 17.3 mm
- net USB_D+: track 0.00 -> 16.9 mm
- net USB_D-: track 0.00 -> 16.6 mm
- net /USB_LDO/RAW_5V: track 0.00 -> 16.2 mm, vias 0 -> 3
- net GND: track 0.00 -> 11.3 mm
- net /USB_LDO/RAW_USB_D-: track 0.00 -> 9.18 mm
- net Net-(J401-CC1): track 0.00 -> 8.40 mm
- net Net-(J401-CC2): track 0.00 -> 8.03 mm
- net /USB_LDO/RAW_USB_D+: track 0.00 -> 7.73 mm
- added copper zone on B.Cu, net GND
- added copper zone on F.Cu, net GND
Other:
- board outline added: 221.5 x 110 mm

Commit message: Tracing 2
Parts:
- added NT201: BAT_0-GND, NetTie:NetTie-2_SMD_Pad0.5mm, F.Cu at (134.5, 117.4)
- moved R703 92.6 mm to (131.4, 62.8), turned to -90 degrees
- moved C702 88.4 mm to (134.5, 62.6), turned to -90 degrees
- moved R702 87.1 mm to (131.4, 67.5), turned to -90 degrees
- moved R701 84.8 mm to (126.9, 65.1), turned to -90 degrees
- moved C701 82.3 mm to (134.5, 67.6), turned to 90 degrees
- moved U701 78.2 mm to (141.7, 65.1), turned to 180 degrees
- moved C803 69.9 mm to (129.7, 82.1)
- moved C802 69.6 mm to (124.5, 82.1), turned to 180 degrees
- moved U601 62.2 mm to (141.7, 54.9)
- moved R603 62.2 mm to (131.4, 52.5), turned to -90 degrees
- moved R601 61.4 mm to (126.9, 54.9), turned to -90 degrees
- moved R602 60.5 mm to (131.4, 57.2), turned to -90 degrees
- moved C602 60.2 mm to (134.5, 52.4)
- moved Q801 60.0 mm to (139.2, 82.8), turned to 180 degrees
- moved C601 59.9 mm to (134.5, 57.4)
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- renumbered J107 to INPUTS, J101 to OUTPUTS
Connections:
- net /Output1/INA226_OUT/VIN+ renamed /Output1/INA226_OUT/VIN
- net /Output2/INA226_OUT/VIN+ renamed /Output2/INA226_OUT/VIN
- net /Output3/INA226_OUT/VIN+ renamed /Output3/INA226_OUT/VIN
- INPUTS pad 1: /INA226_IN/VIN+ -> /INA226_IN/VOUT
- INPUTS pad 2: /INA226_IN/VIN- -> /INA226_IN/VIN
- INPUTS pad 3: /INA226_BAT/VIN+ -> /INA226_BAT/VOUT
- INPUTS pad 4: /INA226_BAT/VIN- -> /INA226_BAT/VIN
- Q1102 pad 2: unconnected-(Q1102-S-Pad2) -> +12V_UPS
- Q1102 pad 3: unconnected-(Q1102-S-Pad3) -> +12V_UPS
- Q802 pad 2: unconnected-(Q802-S-Pad2) -> +12V_UPS
- Q802 pad 3: unconnected-(Q802-S-Pad3) -> +12V_UPS
- Q902 pad 2: unconnected-(Q902-S-Pad2) -> +12V_UPS
- Q902 pad 3: unconnected-(Q902-S-Pad3) -> +12V_UPS
- R601 pad 1: /INA226_IN/VIN- -> /INA226_IN/VOUT
- R601 pad 2: /INA226_IN/VIN+ -> /INA226_IN/VIN
- R602 pad 1: /INA226_IN/VIN+ -> /INA226_IN/VIN
- R603 pad 1: /INA226_IN/VIN- -> /INA226_IN/VOUT
- R701 pad 1: /INA226_BAT/VIN- -> /INA226_BAT/VOUT
- R701 pad 2: /INA226_BAT/VIN+ -> /INA226_BAT/VIN
- R702 pad 1: /INA226_BAT/VIN+ -> /INA226_BAT/VIN
- R703 pad 1: /INA226_BAT/VIN- -> /INA226_BAT/VOUT
- U601 pad 8: /INA226_IN/VIN+ -> /INA226_IN/VIN
- U701 pad 8: /INA226_BAT/VIN+ -> /INA226_BAT/VIN
Routing:
- net +12V_UPS: track 0.00 -> 122.9 mm, vias 0 -> 4
- net +3.3V: track 0.00 -> 44.1 mm
- net /Output1/VOUT: track 0.00 -> 41.0 mm
- net GND: track 11.3 -> 47.8 mm, vias 0 -> 2
- net /INA226_BAT/VIN: track 0.00 -> 32.4 mm, vias 0 -> 2
- net /INA226_IN/VIN: track 0.00 -> 32.4 mm, vias 0 -> 2
- net /Output3/INA226_OUT/VIN: track 0.00 -> 30.7 mm
- net /Output1/INA226_OUT/VIN: track 0.00 -> 28.6 mm, vias 0 -> 2
- net /Output2/INA226_OUT/VIN: track 0.00 -> 28.6 mm, vias 0 -> 2
- net /Output2/VOUT: track 0.00 -> 24.8 mm
- net /Output3/VOUT: track 0.00 -> 23.0 mm
- net /INA226_IN/VOUT: track 0.00 -> 22.9 mm
- net /INA226_BAT/VOUT: track 0.00 -> 22.8 mm
- net Net-(U701-Vin-): track 0.00 -> 10.3 mm
- net Net-(Q902-G): track 0.00 -> 10.2 mm
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Other:
- board size 221.5 x 110 mm -> 105.6 x 87.6 mm
- board text added: "BAT+"
- board text added: "BAT-"
- board text added: "GND"
- board text added: "OUT1"
- board text added: "OUT2"
- board text added: "OUT3"
- board text added: "UPS"
- board text added: "VIN+"
- board text added: "VIN-"

Commit message: Tracing 3
Parts:
- removed C203, C205, C206: 100nF, Capacitor_SMD:C_0603_1608Metric
- removed C204: 1uF, Capacitor_SMD:C_0805_2012Metric
- removed INPUTS: INPUTS, TerminalBlock_Phoenix:TerminalBlock_Phoenix_MKDS-1,5-6-5.08_1x06_P5.08mm_Horizontal
- removed NT201: BAT_0-GND, NetTie:NetTie-2_SMD_Pad0.5mm
- removed OUTPUTS: OUTPUTS, TerminalBlock_Phoenix:TerminalBlock_Phoenix_MKDS-1,5-6-5.08_1x06_P5.08mm_Horizontal
- removed R201: 10K, Resistor_SMD:R_0603_1608Metric_Pad0.98x0.95mm_HandSolder
- removed R202, R203, R204: 200K, Resistor_SMD:R_0603_1608Metric_Pad0.98x0.95mm_HandSolder
- removed R205, R206, R207: 51K, Resistor_SMD:R_0603_1608Metric_Pad0.98x0.95mm_HandSolder
- added CN201: C_Pack04, Resistor_SMD:R_Array_Convex_4x0603, F.Cu at (226.6, 128.0)
- added J101: INPUTS, TerminalBlock_Phoenix:TerminalBlock_Phoenix_MKDS-1,5-6-5.08_1x06_P5.08mm_Horizontal, F.Cu at (112.5, 61.7)
- added J102: OUTPUTS, TerminalBlock_Phoenix:TerminalBlock_Phoenix_MKDS-1,5-6-5.08_1x06_P5.08mm_Horizontal, F.Cu at (112.8, 102.1)
- added J202: BAT_NTC, Connector_JST:JST_GH_SM02B-GHS-TB_1x02-1MP_P1.25mm_Horizontal, F.Cu at (204.7, 126.8)
- added RN201: 39K, Resistor_SMD:R_Array_Convex_4x0603, F.Cu at (202.7, 115.5)
- added RN202: 10K, Resistor_SMD:R_Array_Convex_4x0603, F.Cu at (206.9, 115.5)
- C201: value 100nF -> 1uF; footprint Capacitor_SMD:C_0603_1608Metric -> Capacitor_SMD:C_0805_2012Metric
- J201: footprint Connector_JST:JST_XH_B5B-XH-A_1x05_P2.50mm_Vertical -> Connector_JST:JST_GH_SM04B-GHS-TB_1x04-1MP_P1.25mm_Horizontal
- moved U101 48.9 mm to (237.8, 83.2)
- moved J201 37.2 mm to (191.2, 109.8)
- moved C306 23.4 mm to (148.1, 52.0), turned to 180 degrees
- moved C307 19.0 mm to (148.1, 56.1), turned to 180 degrees
- moved C202 16.3 mm to (166.3, 120.9)
- moved R303 16.0 mm to (148.1, 71.8), turned to 0 degrees
- moved U201 15.8 mm to (183.7, 96.4)
- moved L301 15.8 mm to (157.0, 54.5), turned to 180 degrees
- moved C302 15.4 mm to (148.1, 60.2), turned to 180 degrees
- moved R304 14.1 mm to (147.9, 68.2), turned to 180 degrees
- moved C301 13.6 mm to (148.1, 64.3), turned to 180 degrees
- moved SW101 11.7 mm to (179.9, 110.5)
- moved C304 10.5 mm to (153.6, 71.8), turned to 180 degrees
- moved C401 10.4 mm to (180.1, 61.6)
- moved C402 10.4 mm to (176.2, 67.3)
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Connections:
- C201 pad 1: Net-(U201-AIN0) -> Net-(J202-Pin_2)
- C201 pad 2: BAT_0 -> GND
- C202 pad 1: Net-(U201-AIN1) -> +3.3V
- C202 pad 2: BAT_0 -> GND
- J201 pad 1: BAT_0 -> GND
- U1001 pad 3: unconnected-(U1001-~{Alert}-Pad3) -> /Output2/ALERT
- U1201 pad 3: unconnected-(U1201-~{Alert}-Pad3) -> /Output3/ALERT
- U201 pad 1: BAT_0 -> /BAT_ADS1115/ADDR
- U201 pad 2: unconnected-(U201-ALERT/RDY-Pad2) -> /BAT_ADS1115/ALERT
- U201 pad 3: BAT_0 -> GND
- U201 pad 4: Net-(U201-AIN0) -> Net-(RN201-R1.2)
- U201 pad 5: Net-(U201-AIN1) -> Net-(RN201-R2.2)
- U201 pad 7: Net-(U201-AIN3) -> Net-(J202-Pin_2)
- U201 pad 8: Net-(U201-VDD) -> +3.3V
- U501 pad 3: unconnected-(U501-~{Alert}-Pad3) -> /Output1/ALERT
- U601 pad 3: unconnected-(U601-~{Alert}-Pad3) -> /INA226_IN/ALERT
- U701 pad 3: unconnected-(U701-~{Alert}-Pad3) -> /INA226_BAT/ALERT
Routing:
- net USB_D+: track 16.9 -> 0.00 mm
- net USB_D-: track 16.6 -> 0.74 mm
Other:
- board size 105.6 x 87.6 mm -> 112.8 x 87.6 mm

Commit message: Fixes
Parts:
- CN201: footprint Resistor_SMD:R_Array_Convex_4x0603 -> NosLib:C_Array_Convex_4x0603
- moved U201 38.8 mm to (203.2, 129.9)
- moved CN201 24.0 mm to (203.4, 134.6), turned to -90 degrees
- moved J201 14.1 mm to (192.6, 123.8), turned to -90 degrees
- moved J202 13.3 mm to (192.9, 132.9), turned to -90 degrees
- moved RN201 9.05 mm to (200.8, 124.3)
- moved RN202 8.87 mm to (206.3, 124.3)
- moved U101 4.09 mm to (234.9, 86.0)
Connections:
- U1001 pad 1: GND -> +3.3V
- U1201 pad 1: GND -> SDA
- U201 pad 1: /BAT_ADS1115/ADDR -> GND

Commit message: trace ads1115
Parts:
- removed C202: 100nF, Capacitor_SMD:C_0603_1608Metric
- added R201: 1K, Resistor_SMD:R_0603_1608Metric_Pad0.98x0.95mm_HandSolder, F.Cu at (119.5, 147.1)
- C201: value 1uF -> 100nF; footprint Capacitor_SMD:C_0805_2012Metric -> Capacitor_SMD:C_0603_1608Metric
- CN201: value C_Pack04 -> 100nF
- moved BAT_VOL 87.3 mm to (110.6, 153.8)
- moved RN201 85.9 mm to (119.5, 151.8)
- moved RN202 84.8 mm to (126.1, 151.8)
- moved CN201 84.3 mm to (119.5, 142.5), turned to 180 degrees
- moved BAT_NTC 83.1 mm to (110.6, 143.8)
- moved U201 78.2 mm to (126.1, 142.5)
- moved C201 56.6 mm to (126.2, 147.0), turned to 180 degrees
- moved R103 56.3 mm to (190.3, 82.5)
- moved R104 56.3 mm to (190.3, 85.0)
- moved U101 48.1 mm to (197.8, 116.7), turned to 0 degrees
- moved SW101 7.30 mm to (174.8, 115.7)
- moved C101 6.14 mm to (174.3, 126.2)
- renumbered J202 to BAT_NTC, J201 to BAT_VOL
Connections:
- C201 pad 1: Net-(J202-Pin_2) -> +3.3V
- CN201 pad 1: Net-(RN201-R1.2) -> Net-(U201-AIN3)
- CN201 pad 2: Net-(RN201-R2.2) -> Net-(RN201-R3.2)
- CN201 pad 3: Net-(RN201-R3.2) -> Net-(RN201-R2.2)
- CN201 pad 4: Net-(J202-Pin_2) -> Net-(RN201-R1.2)
- U201 pad 7: Net-(J202-Pin_2) -> Net-(U201-AIN3)
Routing:
- net +3.3V: track 44.1 -> 68.7 mm
- net Net-(RN201-R3.2): track 0.00 -> 23.3 mm, vias 0 -> 2
- net Net-(RN201-R2.2): track 0.00 -> 18.4 mm, vias 0 -> 2
- net Net-(RN201-R1.2): track 0.00 -> 17.6 mm, vias 0 -> 2
- net Net-(J202-Pin_2): track 0.00 -> 17.4 mm, vias 0 -> 2
- net Net-(U201-AIN3): track 0.00 -> 14.3 mm
- net GND: track 47.8 -> 55.6 mm, vias 2 -> 4
- net BAT_3: track 0.00 -> 7.51 mm
- net BAT_2: track 0.00 -> 7.33 mm
- net BAT_1: track 0.00 -> 7.14 mm
Other:
- board size 112.8 x 87.6 mm -> 112.8 x 113.6 mm
