File: hardware/MP2307.kicad_sch (KiCad schematic)
At the start: 17 parts, among them U301 MP2307DN-LF-Z

Commit message: reanotate
Parts:
- renumbered C301 to C901, C302 to C902, C303 to C903, C304 to C904, C305 to C905, C306 to C906, C307 to C907, L301 to L901, NT303 to NT901, NT304 to NT902, NT301 to NT903, NT302 to NT904, R301 to R901, R302 to R902, R303 to R903, R304 to R904, U301 to U901
Changed lines of the file:
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@@
 		(on_board yes)
 		(dnp no)
-		(property "Reference" "C304"
+		(property "Reference" "C904"
 			(at 140.97 96.012 0)
 			(effects
@@
 			(project "NosVolt"
 				(path "/2a3ef4c2-927a-45cd-a4f2-5ee83a7e9444/16799364-b1f1-4a28-ab73-1b10d2d772b3"
-					(reference "C304")
+					(reference "C904")
 					(unit 1)
 				)
@@
 		(dnp no)
 		(fields_autoplaced yes)
-		(property "Reference" "#PWR0301"
+		(property "Reference" "#PWR0903"
 			(at 133.35 119.38 0)
 			(effects
@@
 			(project "NosVolt"
 				(path "/2a3ef4c2-927a-45cd-a4f2-5ee83a7e9444/16799364-b1f1-4a28-ab73-1b10d2d772b3"
-					(reference "#PWR0301")
+					(reference "#PWR0903")
 					(unit 1)
 				)
@@
 		(on_board yes)
 		(dnp no)
-		(property "Reference" "R301"
+		(property "Reference" "R901"
 			(at 114.3 71.374 90)
 			(effects
@@
 			(project "NosVolt"
 				(path "/2a3ef4c2-927a-45cd-a4f2-5ee83a7e9444/16799364-b1f1-4a28-ab73-1b10d2d772b3"
-					(reference "R301")
+					(reference "R901")
 					(unit 1)
 				)
@@
 		(dnp no)
 		(fields_autoplaced yes)
-		(property "Reference" "#PWR0304"
+		(property "Reference" "#PWR0902"
 			(at 128.27 100.33 0)
 			(effects
@@
 			(project "NosVolt"
 				(path "/2a3ef4c2-927a-45cd-a4f2-5ee83a7e9444/16799364-b1f1-4a28-ab73-1b10d2d772b3"
-					(reference "#PWR0304")
+					(reference "#PWR0902")
 					(unit 1)
 				)
@@
 		(dnp no)
 		(fields_autoplaced yes)
-		(property "Reference" "#PWR0303"
+		(property "Reference" "#PWR0901"
 			(at 107.95 119.38 0)
 			(effects
@@
 			(project "NosVolt"
 				(path "/2a3ef4c2-927a-45cd-a4f2-5ee83a7e9444/16799364-b1f1-4a28-ab73-1b10d2d772b3"
-					(reference "#PWR0303")
+					(reference "#PWR0901")
 					(unit 1)
 				)
@@
 		(dnp no)
 		(fields_autoplaced yes)
-		(property "Reference" "C305"
+		(property "Reference" "C905"
 			(at 154.94 68.58 90)
 			(effects
@@
 			(project "NosVolt"
 				(path "/2a3ef4c2-927a-45cd-a4f2-5ee83a7e9444/16799364-b1f1-4a28-ab73-1b10d2d772b3"
-					(reference "C305")
+					(reference "C905")
 					(unit 1)
 				)
@@
 		(on_board yes)
 		(dnp no)
-		(property "Reference" "NT302"
+		(property "Reference" "NT904"
 			(at 175.768 81.788 0)
 			(effects
@@
 			(project "NosVolt"
 				(path "/2a3ef4c2-927a-45cd-a4f2-5ee83a7e9444/16799364-b1f1-4a28-ab73-1b10d2d772b3"
-					(reference "NT302")
+					(reference "NT904")
 					(unit 1)
 				)
@@
 		(dnp no)
 		(fields_autoplaced yes)
-		(property "Reference" "C301"
+		(property "Reference" "C901"
 			(at 82.55 86.3599 0)
 			(effects
@@
 			(project "NosVolt"
 				(path "/2a3ef4c2-927a-45cd-a4f2-5ee83a7e9444/16799364-b1f1-4a28-ab73-1b10d2d772b3"
-					(reference "C301")
+					(reference "C901")
 					(unit 1)
 				)
@@
 		(dnp no)
 		(fields_autoplaced yes)
-		(property "Reference" "L301"
+		(property "Reference" "L901"
 			(at 177.8 71.12 90)
 			(effects
@@
 			(project "NosVolt"
 				(path "/2a3ef4c2-927a-45cd-a4f2-5ee83a7e9444/16799364-b1f1-4a28-ab73-1b10d2d772b3"
-					(reference "L301")
+					(reference "L901")
 					(unit 1)
 				)
@@
 		(on_board yes)
 		(dnp no)
-		(property "Reference" "NT303"
+		(property "Reference" "NT901"
 			(at 99.06 71.374 90)
 			(effects
@@
 			(project ""
 				(path "/2a3ef4c2-927a-45cd-a4f2-5ee83a7e9444/16799364-b1f1-4a28-ab73-1b10d2d772b3"
-					(reference "NT303")
+					(reference "NT901")
 					(unit 1)
 				)
@@
 		(on_board yes)
 		(dnp no)
-		(property "Reference" "R302"
+		(property "Reference" "R902"
 			(at 142.748 105.41 0)
 			(effects
@@
 			(project "NosVolt"
 				(path "/2a3ef4c2-927a-45cd-a4f2-5ee83a7e9444/16799364-b1f1-4a28-ab73-1b10d2d772b3"
-					(reference "R302")
+					(reference "R902")
 					(unit 1)
 				)
@@
 		(on_board yes)
 		(dnp no)
-		(property "Reference" "R303"
+		(property "Reference" "R903"
 			(at 148.082 93.98 0)
 			(effects
@@
 			(project "NosVolt"
 				(path "/2a3ef4c2-927a-45cd-a4f2-5ee83a7e9444/16799364-b1f1-4a28-ab73-1b10d2d772b3"
-					(reference "R303")
+					(reference "R903")
 					(unit 1)
 				)
@@
 		(dnp no)
 		(fields_autoplaced yes)
-		(property "Reference" "#PWR0306"
+		(property "Reference" "#PWR0905"
 			(at 152.4 119.38 0)
 			(effects
@@
 			(project "NosVolt"
 				(path "/2a3ef4c2-927a-45cd-a4f2-5ee83a7e9444/16799364-b1f1-4a28-ab73-1b10d2d772b3"
-					(reference "#PWR0306")
+					(reference "#PWR0905")
 					(unit 1)
 				)
@@
 		(on_board yes)
 		(dnp no)
-		(property "Reference" "NT304"
+		(property "Reference" "NT902"
 			(at 125.476 106.934 90)
 			(effects
@@
 			(project "NosVolt"
 				(path "/2a3ef4c2-927a-45cd-a4f2-5ee83a7e9444/16799364-b1f1-4a28-ab73-1b10d2d772b3"
-					(reference "NT304")
+					(reference "NT902")
 					(unit 1)
 				)
@@
 		(dnp no)
 		(fields_autoplaced yes)
-		(property "Reference" "C302"
+		(property "Reference" "C902"
 			(at 93.98 86.3599 0)
 			(effects
@@
 			(project "NosVolt"
 				(path "/2a3ef4c2-927a-45cd-a4f2-5ee83a7e9444/16799364-b1f1-4a28-ab73-1b10d2d772b3"
-					(reference "C302")
+					(reference "C902")
 					(unit 1)
 				)
@@
 		(dnp no)
 		(fields_autoplaced yes)
-		(property "Reference" "#PWR0305"
+		(property "Reference" "#PWR0904"
 			(at 138.43 119.38 0)
 			(effects
@@
 			(project "NosVolt"
 				(path "/2a3ef4c2-927a-45cd-a4f2-5ee83a7e9444/16799364-b1f1-4a28-ab73-1b10d2d772b3"
-					(reference "#PWR0305")
+					(reference "#PWR0904")
 					(unit 1)
 				)
@@
 		(dnp no)
 		(fields_autoplaced yes)
-		(property "Reference" "C307"
+		(property "Reference" "C907"
 			(at 210.82 91.4399 0)
 			(effects
@@
 			(project "NosVolt"
 				(path "/2a3ef4c2-927a-45cd-a4f2-5ee83a7e9444/16799364-b1f1-4a28-ab73-1b10d2d772b3"
-					(reference "C307")
+					(reference "C907")
 					(unit 1)
 				)
@@
 		(dnp no)
 		(fields_autoplaced yes)
-		(property "Reference" "C303"
+		(property "Reference" "C903"
 			(at 111.76 95.2499 0)
 			(effects
@@
 			(project "NosVolt"
 				(path "/2a3ef4c2-927a-45cd-a4f2-5ee83a7e9444/16799364-b1f1-4a28-ab73-1b10d2d772b3"
-					(reference "C303")
+					(reference "C903")
 					(unit 1)
 				)
@@
 		(on_board yes)
 		(dnp no)
-		(property "Reference" "C306"
+		(property "Reference" "C906"
 			(at 191.77 91.4399 0)
 			(effects
@@
 			(project "NosVolt"
 				(path "/2a3ef4c2-927a-45cd-a4f2-5ee83a7e9444/16799364-b1f1-4a28-ab73-1b10d2d772b3"
-					(reference "C306")
+					(reference "C906")
 					(unit 1)
 				)
@@
 		(on_board yes)
 		(dnp no)
-		(property "Reference" "U301"
+		(property "Reference" "U901"
 			(at 135.128 67.564 0)
 			(effects
@@
 			(project "NosVolt"
 				(path "/2a3ef4c2-927a-45cd-a4f2-5ee83a7e9444/16799364-b1f1-4a28-ab73-1b10d2d772b3"
-					(reference "U301")
+					(reference "U901")
 					(unit 1)
 				)
@@
 		(on_board yes)
 		(dnp no)
-		(property "Reference" "NT301"
+		(property "Reference" "NT903"
 			(at 164.338 70.612 0)
 			(effects
@@
 			(project ""
 				(path "/2a3ef4c2-927a-45cd-a4f2-5ee83a7e9444/16799364-b1f1-4a28-ab73-1b10d2d772b3"
-					(reference "NT301")
+					(reference "NT903")
 					(unit 1)
 				)
@@
 		(on_board yes)
 		(dnp no)
-		(property "Reference" "R304"
+		(property "Reference" "R904"
 			(at 160.274 86.36 90)
 			(effects
@@
 			(project "NosVolt"
 				(path "/2a3ef4c2-927a-45cd-a4f2-5ee83a7e9444/16799364-b1f1-4a28-ab73-1b10d2d772b3"
-					(reference "R304")
-					(unit 1)
-				)
+					(reference "R904")
+					(unit 1)
+				)
