File: hardware/USB_LDO.kicad_sch (KiCad schematic)
At the start: 12 parts, among them J1 USB_C_Receptacle_USB2.0_16P, U2 AP7361-33ER-13, U6 USBLC6-2SC6

Commit message: Outputs and current measurement
Parts:
- R401: renamed from R5; footprint Resistor_SMD:R_0603_1608Metric -> Resistor_SMD:R_0603_1608Metric_Pad0.98x0.95mm_HandSolder
- R402: renamed from R6; footprint Resistor_SMD:R_0603_1608Metric -> Resistor_SMD:R_0603_1608Metric_Pad0.98x0.95mm_HandSolder
- renumbered C1 to C401, C3 to C402, C4 to C403, C5 to C404, C6 to C405, D1 to D401, F1 to F401, J1 to J401, U2 to U401, U6 to U402
Changed lines of the file:
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@@
+	(wire
+		(pts
+			(xy 77.47 138.43) (xy 86.36 138.43)
+		)
+		(stroke
+			(width 0)
+			(type default)
+		)
+	)
 	(wire
 		(pts
@@
 	(wire
 		(pts
-			(xy 114.3 97.79) (xy 134.62 97.79)
+			(xy 109.22 97.79) (xy 134.62 97.79)
 		)
 		(stroke
@@
 	(wire
 		(pts
-			(xy 111.76 100.33) (xy 111.76 99.06)
+			(xy 106.68 100.33) (xy 106.68 99.06)
 		)
 		(stroke
@@
 	(wire
 		(pts
-			(xy 81.28 138.43) (xy 86.36 138.43)
-		)
-		(stroke
-			(width 0)
-			(type default)
-		)
-	)
-	(wire
-		(pts
 			(xy 120.65 86.36) (xy 120.65 90.17)
 		)
@@
 	(wire
 		(pts
-			(xy 106.68 93.98) (xy 114.3 93.98)
+			(xy 106.68 93.98) (xy 109.22 93.98)
 		)
 		(stroke
@@
 	(wire
 		(pts
-			(xy 114.3 93.98) (xy 114.3 97.79)
+			(xy 109.22 93.98) (xy 109.22 97.79)
 		)
 		(stroke
@@
 	(wire
 		(pts
-			(xy 111.76 99.06) (xy 106.68 99.06)
-		)
-		(stroke
-			(width 0)
-			(type default)
-		)
-	)
-	(wire
-		(pts
 			(xy 86.36 138.43) (xy 101.6 138.43)
 		)
@@
 	(wire
 		(pts
-			(xy 134.62 100.33) (xy 111.76 100.33)
+			(xy 134.62 100.33) (xy 106.68 100.33)
 		)
 		(stroke
@@
 	(wire
 		(pts
-			(xy 139.7 78.74) (xy 146.05 78.74)
-		)
-		(stroke
-			(width 0)
-			(type default)
-		)
-	)
-	(wire
-		(pts
 			(xy 101.6 138.43) (xy 107.95 138.43)
 		)
@@
 			(width 0)
 			(type default)
-		)
-	)
-	(label "5V"
-		(at 81.28 138.43 0)
-		(effects
-			(font
-				(size 1.27 1.27)
-			)
-			(justify left bottom)
-		)
-	)
-	(label "5V"
-		(at 146.05 78.74 0)
-		(effects
-			(font
-				(size 1.27 1.27)
-			)
-			(justify left bottom)
 		)
 	)
@@
 			)
 			(justify left)
+		)
+	)
+	(hierarchical_label "5V"
+		(shape output)
+		(at 77.47 138.43 180)
+		(effects
+			(font
+				(size 1.27 1.27)
+			)
+			(justify right)
 		)
 	)
@@
 		(dnp no)
 		(fields_autoplaced yes)
-		(property "Reference" "#PWR07"
+		(property "Reference" "#PWR0403"
 			(at 120.65 96.52 0)
 			(effects
@@
 			(project ""
 				(path "/2a3ef4c2-927a-45cd-a4f2-5ee83a7e9444/a3c788b2-be52-41e3-a33a-7de63687b368"
-					(reference "#PWR07")
+					(reference "#PWR0403")
 					(unit 1)
 				)
@@
 		(dnp no)
 		(fields_autoplaced yes)
-		(property "Reference" "C6"
+		(property "Reference" "C405"
 			(at 143.51 143.5099 0)
 			(effects
@@
 			(project "NosVolt"
 				(path "/2a3ef4c2-927a-45cd-a4f2-5ee83a7e9444/a3c788b2-be52-41e3-a33a-7de63687b368"
-					(reference "C6")
+					(reference "C405")
 					(unit 1)
 				)
@@
 		(on_board yes)
 		(dnp no)
-		(property "Reference" "J1"
+		(property "Reference" "J401"
 			(at 90.17 71.12 0)
 			(effects
@@
 			(project "NosVolt"
 				(path "/2a3ef4c2-927a-45cd-a4f2-5ee83a7e9444/a3c788b2-be52-41e3-a33a-7de63687b368"
-					(reference "J1")
+					(reference "J401")
 					(unit 1)
 				)
@@
 		(on_board yes)
 		(dnp no)
-		(property "Reference" "U6"
+		(property "Reference" "U402"
 			(at 142.8181 107.95 0)
 			(effects
@@
 			(project "NosVolt"
 				(path "/2a3ef4c2-927a-45cd-a4f2-5ee83a7e9444/a3c788b2-be52-41e3-a33a-7de63687b368"
-					(reference "U6")
+					(reference "U402")
 					(unit 1)
 				)
@@
 		(dnp no)
 		(fields_autoplaced yes)
-		(property "Reference" "C5"
+		(property "Reference" "C404"
 			(at 129.54 143.5099 0)
 			(effects
@@
 			(project "NosVolt"
 				(path "/2a3ef4c2-927a-45cd-a4f2-5ee83a7e9444/a3c788b2-be52-41e3-a33a-7de63687b368"
-					(reference "C5")
+					(reference "C404")
 					(unit 1)
 				)
@@
 		(dnp no)
 		(fields_autoplaced yes)
-		(property "Reference" "#PWR010"
+		(property "Reference" "#PWR0402"
 			(at 115.57 161.29 0)
 			(effects
@@
 			(project "NosVolt"
 				(path "/2a3ef4c2-927a-45cd-a4f2-5ee83a7e9444/a3c788b2-be52-41e3-a33a-7de63687b368"
-					(reference "#PWR010")
+					(reference "#PWR0402")
 					(unit 1)
 				)
@@
 		(dnp no)
 		(fields_autoplaced yes)
-		(property "Reference" "#PWR021"
+		(property "Reference" "#PWR0405"
 			(at 139.7 111.76 0)
 			(effects
@@
 			(project "NosVolt"
 				(path "/2a3ef4c2-927a-45cd-a4f2-5ee83a7e9444/a3c788b2-be52-41e3-a33a-7de63687b368"
-					(reference "#PWR021")
+					(reference "#PWR0405")
 					(unit 1)
 				)
@@
 		(dnp no)
 		(fields_autoplaced yes)
-		(property "Reference" "U2"
+		(property "Reference" "U401"
 			(at 115.57 132.08 0)
 			(effects
@@
 			(project "NosVolt"
 				(path "/2a3ef4c2-927a-45cd-a4f2-5ee83a7e9444/a3c788b2-be52-41e3-a33a-7de63687b368"
-					(reference "U2")
+					(reference "U401")
 					(unit 1)
 				)
@@
 		(on_board yes)
 		(dnp no)
-		(property "Reference" "R6"
-			(at 110.236 88.646 90)
+		(property "Reference" "R402"
+			(at 109.474 88.646 90)
 			(effects
 				(font
@@
 		)
 		(property "Value" "5.1K"
-			(at 114.3 88.646 90)
-			(effects
-				(font
-					(size 1.27 1.27)
-				)
-			)
-		)
-		(property "Footprint" "Resistor_SMD:R_0603_1608Metric"
+			(at 115.824 88.646 90)
+			(effects
+				(font
+					(size 1.27 1.27)
+				)
+			)
+		)
+		(property "Footprint" "Resistor_SMD:R_0603_1608Metric_Pad0.98x0.95mm_HandSolder"
 			(at 111.76 88.138 90)
 			(effects
@@
 			(project "NosVolt"
 				(path "/2a3ef4c2-927a-45cd-a4f2-5ee83a7e9444/a3c788b2-be52-41e3-a33a-7de63687b368"
-					(reference "R6")
+					(reference "R402")
 					(unit 1)
 				)
@@
 		(on_board yes)
 		(dnp no)
-		(property "Reference" "C1"
+		(property "Reference" "C401"
 			(at 76.2 118.11 0)
 			(effects
@@
 			(project "NosVolt"
 				(path "/2a3ef4c2-927a-45cd-a4f2-5ee83a7e9444/a3c788b2-be52-41e3-a33a-7de63687b368"
-					(reference "C1")
+					(reference "C401")
 					(unit 1)
 				)
@@
 		(dnp no)
 		(fields_autoplaced yes)
-		(property "Reference" "#PWR08"
+		(property "Reference" "#PWR0404"
 			(at 125.73 96.52 0)
 			(effects
@@
 			(project ""
 				(path "/2a3ef4c2-927a-45cd-a4f2-5ee83a7e9444/a3c788b2-be52-41e3-a33a-7de63687b368"
-					(reference "#PWR08")
+					(reference "#PWR0404")
 					(unit 1)
 				)
@@
 		(on_board yes)
 		(dnp no)
-		(property "Reference" "F1"
+		(property "Reference" "F401"
 			(at 112.014 72.136 90)
 			(effects
@@
 			(project "NosVolt"
 				(path "/2a3ef4c2-927a-45cd-a4f2-5ee83a7e9444/a3c788b2-be52-41e3-a33a-7de63687b368"
-					(reference "F1")
+					(reference "F401")
 					(unit 1)
 				)
@@
 		(dnp no)
 		(fields_autoplaced yes)
-		(property "Reference" "C4"
+		(property "Reference" "C403"
 			(at 105.41 143.5099 0)
 			(effects
@@
 			(project "NosVolt"
 				(path "/2a3ef4c2-927a-45cd-a4f2-5ee83a7e9444/a3c788b2-be52-41e3-a33a-7de63687b368"
-					(reference "C4")
+					(reference "C403")
 					(unit 1)
 				)
@@
 		(dnp no)
 		(fields_autoplaced yes)
-		(property "Reference" "D1"
+		(property "Reference" "D401"
 			(at 128.27 83.8199 90)
 			(effects
@@
 			(project "NosVolt"
 				(path "/2a3ef4c2-927a-45cd-a4f2-5ee83a7e9444/a3c788b2-be52-41e3-a33a-7de63687b368"
-					(reference "D1")
+					(reference "D401")
 					(unit 1)
 				)
@@
 		(dnp no)
 		(fields_autoplaced yes)
-		(property "Reference" "#PWR09"
+		(property "Reference" "#PWR0401"
 			(at 90.17 133.35 0)
 			(effects
@@
 			(project "NosVolt"
 				(path "/2a3ef4c2-927a-45cd-a4f2-5ee83a7e9444/a3c788b2-be52-41e3-a33a-7de63687b368"
-					(reference "#PWR09")
+					(reference "#PWR0401")
 					(unit 1)
 				)
@@
 		(dnp no)
 		(fields_autoplaced yes)
-		(property "Reference" "C3"
+		(property "Reference" "C402"
 			(at 90.17 143.5099 0)
 			(effects
@@
 			(project "NosVolt"
 				(path "/2a3ef4c2-927a-45cd-a4f2-5ee83a7e9444/a3c788b2-be52-41e3-a33a-7de63687b368"
-					(reference "C3")
+					(reference "C402")
 					(unit 1)
 				)
@@
 		(on_board yes)
 		(dnp no)
-		(property "Reference" "R5"
-			(at 109.982 81.534 90)
+		(property "Reference" "R401"
+			(at 109.474 81.534 90)
 			(effects
 				(font
@@
 		)
 		(property "Value" "5.1K"
-			(at 113.792 81.534 90)
-			(effects
-				(font
-					(size 1.27 1.27)
-				)
-			)
-		)
-		(property "Footprint" "Resistor_SMD:R_0603_1608Metric"
+			(at 115.824 81.534 90)
+			(effects
+				(font
+					(size 1.27 1.27)
+				)
+			)
+		)
+		(property "Footprint" "Resistor_SMD:R_0603_1608Metric_Pad0.98x0.95mm_HandSolder"
 			(at 111.76 85.598 90)
 			(effects
@@
 			(project "NosVolt"
 				(path "/2a3ef4c2-927a-45cd-a4f2-5ee83a7e9444/a3c788b2-be52-41e3-a33a-7de63687b368"
-					(reference "R5")
+					(reference "R401")
 					(unit 1)
 				)

Commit message: Tracing 1
Connections:
- net DM: now also U402.6 (I/O1); no longer U402.1 (I/O1)
- net DP: now also U402.4 (I/O2); no longer U402.3 (I/O2)
- net RAW_5V: now reaches F401.1, J401.A4 (VBUS), J401.A9 (VBUS), J401.B4 (VBUS), J401.B9 (VBUS)
- net RAW_USB_D+: now reaches J401.A6 (D+), J401.B6 (D+)
- net RAW_USB_D+: now also U402.3 (I/O2); no longer U402.4 (I/O2)
- net RAW_USB_D-: now reaches J401.A7 (D-), J401.B7 (D-)
- net RAW_USB_D-: now also U402.1 (I/O1); no longer U402.6 (I/O1)
Other:
- moved on the sheet: F401, U402
Changed lines of the file:
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@@
+	)
+	(junction
+		(at 125.73 78.74)
+		(diameter 0)
+		(color 0 0 0 0)
 	)
 	(junction
@@
 	)
 	(junction
-		(at 125.73 78.74)
-		(diameter 0)
-		(color 0 0 0 0)
-	)
-	(junction
 		(at 120.65 86.36)
 		(diameter 0)
@@
 	(wire
 		(pts
-			(xy 139.7 78.74) (xy 139.7 92.71)
-		)
-		(stroke
-			(width 0)
-			(type default)
-		)
-	)
-	(wire
-		(pts
-			(xy 109.22 97.79) (xy 134.62 97.79)
+			(xy 109.22 101.6) (xy 134.62 101.6)
 		)
 		(stroke
@@
 	(wire
 		(pts
-			(xy 106.68 100.33) (xy 106.68 99.06)
+			(xy 106.68 104.14) (xy 106.68 99.06)
 		)
 		(stroke
@@
 	(wire
 		(pts
+			(xy 139.7 78.74) (xy 139.7 96.52)
+		)
+		(stroke
+			(width 0)
+			(type default)
+		)
+	)
+	(wire
+		(pts
 			(xy 106.68 96.52) (xy 106.68 99.06)
 		)
@@
 	(wire
 		(pts
-			(xy 115.57 78.74) (xy 125.73 78.74)
-		)
-		(stroke
-			(width 0)
-			(type default)
-		)
-	)
-	(wire
-		(pts
 			(xy 106.68 91.44) (xy 106.68 93.98)
 		)
@@
 	(wire
 		(pts
+			(xy 123.19 78.74) (xy 125.73 78.74)
+		)
+		(stroke
+			(width 0)
+			(type default)
+		)
+	)
+	(wire
+		(pts
 			(xy 90.17 124.46) (xy 90.17 127)
 		)
@@
 	(wire
 		(pts
-			(xy 109.22 93.98) (xy 109.22 97.79)
+			(xy 139.7 78.74) (xy 125.73 78.74)
+		)
+		(stroke
+			(width 0)
+			(type default)
+		)
+	)
+	(wire
+		(pts
+			(xy 109.22 93.98) (xy 109.22 101.6)
 		)
 		(stroke
@@
 	(wire
 		(pts
+			(xy 105.41 78.74) (xy 115.57 78.74)
+		)
+		(stroke
+			(width 0)
+			(type default)
+		)
+	)
+	(wire
+		(pts
 			(xy 90.17 116.84) (xy 90.17 124.46)
 		)
@@
 	(wire
 		(pts
+			(xy 153.67 101.6) (xy 144.78 101.6)
+		)
+		(stroke
+			(width 0)
+			(type default)
+		)
+	)
+	(wire
+		(pts
 			(xy 115.57 151.13) (xy 125.73 151.13)
 		)
@@
 	(wire
 		(pts
-			(xy 125.73 78.74) (xy 139.7 78.74)
-		)
-		(stroke
-			(width 0)
-			(type default)
-		)
-	)
-	(wire
-		(pts
 			(xy 115.57 151.13) (xy 115.57 154.94)
 		)
@@
 	(wire
 		(pts
-			(xy 134.62 100.33) (xy 106.68 100.33)
+			(xy 134.62 104.14) (xy 106.68 104.14)
+		)
+		(stroke
+			(width 0)
+			(type default)
+		)
+	)
+	(wire
+		(pts
+			(xy 153.67 104.14) (xy 144.78 104.14)
 		)
 		(stroke
@@
 	(wire
 		(pts
-			(xy 105.41 78.74) (xy 107.95 78.74)
-		)
-		(stroke
-			(width 0)
-			(type default)
-		)
-	)
-	(wire
-		(pts
 			(xy 106.68 91.44) (xy 105.41 91.44)
 		)
@@
 			(width 0)
 			(type default)
+		)
+	)
+	(label "USB_D-"
+		(at 146.05 101.6 0)
+		(effects
+			(font
+				(size 1.27 1.27)
+			)
+			(justify left bottom)
+		)
+	)
+	(label "RAW_5V"
+		(at 105.41 78.74 0)
+		(effects
+			(font
+				(size 1.27 1.27)
+			)
+			(justify left bottom)
+		)
+	)
+	(label "RAW_USB_D-"
+		(at 113.03 101.6 0)
+		(effects
+			(font
+				(size 1.27 1.27)
+			)
+			(justify left bottom)
+		)
+	)
+	(label "RAW_USB_D+"
+		(at 113.03 104.14 0)
+		(effects
+			(font
+				(size 1.27 1.27)
+			)
+			(justify left bottom)
+		)
+	)
+	(label "USB_D+"
+		(at 146.05 104.14 0)
+		(effects
+			(font
+				(size 1.27 1.27)
+			)
+			(justify left bottom)
 		)
 	)
@@
 	(hierarchical_label "DP"
 		(shape bidirectional)
-		(at 144.78 100.33 0)
+		(at 153.67 104.14 0)
 		(effects
 			(font
@@
 	(hierarchical_label "DM"
 		(shape bidirectional)
-		(at 144.78 97.79 0)
+		(at 153.67 101.6 0)
 		(effects
 			(font
@@
 	(symbol
 		(lib_id "Power_Protection:USBLC6-2SC6")
-		(at 139.7 97.79 0)
-		(mirror y)
+		(at 139.7 101.6 0)
 		(unit 1)
 		(exclude_from_sim no)
@@
 		(dnp no)
 		(property "Reference" "U402"
-			(at 142.8181 107.95 0)
+			(at 136.5819 111.76 0)
 			(effects
 				(font
@@
 		)
 		(property "Value" "USBLC6-2SC6"
-			(at 142.748 105.156 0)
+			(at 136.652 108.966 0)
 			(effects
 				(font
@@
 		)
 		(property "Footprint" "Package_TO_SOT_SMD:SOT-23-6"
-			(at 138.43 104.14 0)
+			(at 140.97 107.95 0)
 			(effects
 				(font
@@
 		)
 		(property "Datasheet" "https://www.st.com/resource/en/datasheet/usblc6-2.pdf"
-			(at 138.43 106.045 0)
+			(at 140.97 109.855 0)
 			(effects
 				(font
@@
 		)
 		(property "Description" "Very low capacitance ESD protection diode, 2 data-line, SOT-23-6"
-			(at 139.7 97.79 0)
+			(at 139.7 101.6 0)
 			(effects
 				(font
@@
 	(symbol
 		(lib_id "power:GND")
-		(at 139.7 105.41 0)
+		(at 139.7 109.22 0)
 		(unit 1)
 		(exclude_from_sim no)
@@
 		(fields_autoplaced yes)
 		(property "Reference" "#PWR0405"
-			(at 139.7 111.76 0)
+			(at 139.7 115.57 0)
 			(effects
 				(font
@@
 		)
 		(property "Value" "GND"
-			(at 139.7 110.49 0)
+			(at 139.7 114.3 0)
 			(effects
 				(font
@@
 		)
 		(property "Footprint" ""
-			(at 139.7 105.41 0)
+			(at 139.7 109.22 0)
 			(effects
 				(font
@@
 		)
 		(property "Datasheet" ""
-			(at 139.7 105.41 0)
+			(at 139.7 109.22 0)
 			(effects
 				(font
@@
 		)
 		(property "Description" "Power symbol creates a global label with name \"GND\" , ground"
-			(at 139.7 105.41 0)
+			(at 139.7 109.22 0)
 			(effects
 				(font
@@
 	(symbol
 		(lib_id "Device:Polyfuse")
-		(at 111.76 78.74 90)
+		(at 119.38 78.74 90)
 		(unit 1)
 		(exclude_from_sim no)
@@
 		(dnp no)
 		(property "Reference" "F401"
-			(at 112.014 72.136 90)
+			(at 119.634 72.136 90)
 			(effects
 				(font
@@
 		)
 		(property "Value" "Polyfuse 0.75A"
-			(at 111.76 74.93 90)
+			(at 119.38 74.93 90)
 			(effects
 				(font
@@
 		)
 		(property "Footprint" "Fuse:Fuse_0805_2012Metric"
-			(at 116.84 77.47 0)
+			(at 124.46 77.47 0)
 			(effects
 				(font
@@
 		)
 		(property "Datasheet" "~"
-			(at 111.76 78.74 0)
+			(at 119.38 78.74 0)
 			(effects
 				(font
@@
 		)
 		(property "Description" "Resettable fuse, polymeric positive temperature coefficient"
-			(at 111.76 78.74 0)
-			(effects
-				(font
+			(at 119.38 78.74 0)
+			(effects
+				(font

Commit message: Add screen
Connections:
- net 3V3 renamed USB_3V3
- net 5V renamed USB_5V
Changed lines of the file:
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@@
 		)
 	)
-	(hierarchical_label "5V"
+	(hierarchical_label "USB_5V"
 		(shape output)
 		(at 139.7 69.85 90)
@@
 		)
 	)
-	(hierarchical_label "5V"
+	(hierarchical_label "USB_5V"
 		(shape output)
 		(at 77.47 138.43 180)
@@
 		)
 	)
-	(hierarchical_label "3V3"
+	(hierarchical_label "USB_3V3"
 		(shape output)
 		(at 149.86 138.43 0)
@@
 		)
 		(instances
-			(project ""
-				(path "/2a3ef4c2-927a-45cd-a4f2-5ee83a7e9444/a3c788b2-be52-41e3-a33a-7de63687b368"
+			(project "NosVolt"
+				(path "/2a3ef4c2-927a-45cd-a4f2-5ee83a7e9444/f9001ea6-7fd9-45f8-b2c2-99ce1a63a0f2"
 					(reference "#PWR0403")
 					(unit 1)
@@
 		(instances
 			(project "NosVolt"
-				(path "/2a3ef4c2-927a-45cd-a4f2-5ee83a7e9444/a3c788b2-be52-41e3-a33a-7de63687b368"
+				(path "/2a3ef4c2-927a-45cd-a4f2-5ee83a7e9444/f9001ea6-7fd9-45f8-b2c2-99ce1a63a0f2"
 					(reference "C405")
 					(unit 1)
@@
 		(instances
 			(project "NosVolt"
-				(path "/2a3ef4c2-927a-45cd-a4f2-5ee83a7e9444/a3c788b2-be52-41e3-a33a-7de63687b368"
+				(path "/2a3ef4c2-927a-45cd-a4f2-5ee83a7e9444/f9001ea6-7fd9-45f8-b2c2-99ce1a63a0f2"
 					(reference "J401")
 					(unit 1)
@@
 		(instances
 			(project "NosVolt"
-				(path "/2a3ef4c2-927a-45cd-a4f2-5ee83a7e9444/a3c788b2-be52-41e3-a33a-7de63687b368"
+				(path "/2a3ef4c2-927a-45cd-a4f2-5ee83a7e9444/f9001ea6-7fd9-45f8-b2c2-99ce1a63a0f2"
 					(reference "U402")
 					(unit 1)
@@
 		(instances
 			(project "NosVolt"
-				(path "/2a3ef4c2-927a-45cd-a4f2-5ee83a7e9444/a3c788b2-be52-41e3-a33a-7de63687b368"
+				(path "/2a3ef4c2-927a-45cd-a4f2-5ee83a7e9444/f9001ea6-7fd9-45f8-b2c2-99ce1a63a0f2"
 					(reference "C404")
 					(unit 1)
@@
 		(instances
 			(project "NosVolt"
-				(path "/2a3ef4c2-927a-45cd-a4f2-5ee83a7e9444/a3c788b2-be52-41e3-a33a-7de63687b368"
+				(path "/2a3ef4c2-927a-45cd-a4f2-5ee83a7e9444/f9001ea6-7fd9-45f8-b2c2-99ce1a63a0f2"
 					(reference "#PWR0402")
 					(unit 1)
@@
 		(instances
 			(project "NosVolt"
-				(path "/2a3ef4c2-927a-45cd-a4f2-5ee83a7e9444/a3c788b2-be52-41e3-a33a-7de63687b368"
+				(path "/2a3ef4c2-927a-45cd-a4f2-5ee83a7e9444/f9001ea6-7fd9-45f8-b2c2-99ce1a63a0f2"
 					(reference "#PWR0405")
 					(unit 1)
@@
 		(instances
 			(project "NosVolt"
-				(path "/2a3ef4c2-927a-45cd-a4f2-5ee83a7e9444/a3c788b2-be52-41e3-a33a-7de63687b368"
+				(path "/2a3ef4c2-927a-45cd-a4f2-5ee83a7e9444/f9001ea6-7fd9-45f8-b2c2-99ce1a63a0f2"
 					(reference "U401")
 					(unit 1)
@@
 		(instances
 			(project "NosVolt"
-				(path "/2a3ef4c2-927a-45cd-a4f2-5ee83a7e9444/a3c788b2-be52-41e3-a33a-7de63687b368"
+				(path "/2a3ef4c2-927a-45cd-a4f2-5ee83a7e9444/f9001ea6-7fd9-45f8-b2c2-99ce1a63a0f2"
 					(reference "R402")
 					(unit 1)
@@
 		(instances
 			(project "NosVolt"
-				(path "/2a3ef4c2-927a-45cd-a4f2-5ee83a7e9444/a3c788b2-be52-41e3-a33a-7de63687b368"
+				(path "/2a3ef4c2-927a-45cd-a4f2-5ee83a7e9444/f9001ea6-7fd9-45f8-b2c2-99ce1a63a0f2"
 					(reference "C401")
 					(unit 1)
@@
 		)
 		(instances
-			(project ""
-				(path "/2a3ef4c2-927a-45cd-a4f2-5ee83a7e9444/a3c788b2-be52-41e3-a33a-7de63687b368"
+			(project "NosVolt"
+				(path "/2a3ef4c2-927a-45cd-a4f2-5ee83a7e9444/f9001ea6-7fd9-45f8-b2c2-99ce1a63a0f2"
 					(reference "#PWR0404")
 					(unit 1)
@@
 		(instances
 			(project "NosVolt"
-				(path "/2a3ef4c2-927a-45cd-a4f2-5ee83a7e9444/a3c788b2-be52-41e3-a33a-7de63687b368"
+				(path "/2a3ef4c2-927a-45cd-a4f2-5ee83a7e9444/f9001ea6-7fd9-45f8-b2c2-99ce1a63a0f2"
 					(reference "F401")
 					(unit 1)
@@
 		(instances
 			(project "NosVolt"
-				(path "/2a3ef4c2-927a-45cd-a4f2-5ee83a7e9444/a3c788b2-be52-41e3-a33a-7de63687b368"
+				(path "/2a3ef4c2-927a-45cd-a4f2-5ee83a7e9444/f9001ea6-7fd9-45f8-b2c2-99ce1a63a0f2"
 					(reference "C403")
 					(unit 1)
@@
 		(instances
 			(project "NosVolt"
-				(path "/2a3ef4c2-927a-45cd-a4f2-5ee83a7e9444/a3c788b2-be52-41e3-a33a-7de63687b368"
+				(path "/2a3ef4c2-927a-45cd-a4f2-5ee83a7e9444/f9001ea6-7fd9-45f8-b2c2-99ce1a63a0f2"
 					(reference "D401")
 					(unit 1)
@@
 		(instances
 			(project "NosVolt"
-				(path "/2a3ef4c2-927a-45cd-a4f2-5ee83a7e9444/a3c788b2-be52-41e3-a33a-7de63687b368"
+				(path "/2a3ef4c2-927a-45cd-a4f2-5ee83a7e9444/f9001ea6-7fd9-45f8-b2c2-99ce1a63a0f2"
 					(reference "#PWR0401")
 					(unit 1)
@@
 		(instances
 			(project "NosVolt"
-				(path "/2a3ef4c2-927a-45cd-a4f2-5ee83a7e9444/a3c788b2-be52-41e3-a33a-7de63687b368"
+				(path "/2a3ef4c2-927a-45cd-a4f2-5ee83a7e9444/f9001ea6-7fd9-45f8-b2c2-99ce1a63a0f2"
 					(reference "C402")
 					(unit 1)
@@
 		(instances
 			(project "NosVolt"
-				(path "/2a3ef4c2-927a-45cd-a4f2-5ee83a7e9444/a3c788b2-be52-41e3-a33a-7de63687b368"
+				(path "/2a3ef4c2-927a-45cd-a4f2-5ee83a7e9444/f9001ea6-7fd9-45f8-b2c2-99ce1a63a0f2"
 					(reference "R401")
 					(unit 1)
